File: Hardware/RedBot Accelerometer.sch (EAGLE design)
At the start: 20 parts, among them Q1 220mA/50V/3.5Ω, Q2 220mA/50V/3.5Ω, U1 MMA8452QMMA8452Q-1:1, U2 MIC5205-3.3V

Commit message: updating old packages
Parts:
- added LOGO4: SFE_LOGO_FLAME.1_INCH, SparkFun-Aesthetics:SFE_LOGO_FLAME.1_INCH
- C1, C3: device SparkFun-Capacitors:0.1UF-25V(+80/-20%)(0603) -> SparkFun-Capacitors:0.1UF-0603-25V-(+80/-20%)
- C2: device SparkFun-Capacitors:4.7UF-6.3V-10%(0603)0603 -> SparkFun-Capacitors:4.7UF-0603-6.3V-(10%)
- R1: device SparkFun-Resistors:10KOHM1/10W1%(0603)0603 -> SparkFun-Resistors:10KOHM-0603-1/10W-1%
- U1: value MMA8452QMMA8452Q-1:1 -> MMA8452Q; device SparkFun-Sensors:MMA8452QMMA8452Q-1:1 -> SparkFun-Sensors:MMA8452Q
Connections:
- net 3.3V: no longer U1.VDDIO
- net GND: now also U1.GND; no longer U1.GND@0, U1.GND@1, U1.GND@2
Other:
- note added: "7-bit Unshifted I2C Address: 0x1D"
- note added: "VIN: 2.5-16V"
Changed lines of the file:
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@@
 <part name="LOGO1" library="SparkFun-Aesthetics" deviceset="LOGO-SFE" device="SK"/>
 <part name="LOGO2" library="SparkFun-Aesthetics" deviceset="OSHW-LOGO" device="S"/>
-<part name="C1" library="SparkFun-Capacitors" deviceset="0.1UF-25V(+80/-20%)(0603)" device="" value="0.1uF"/>
-<part name="U1" library="SparkFun-Sensors" deviceset="MMA8452Q" device="MMA8452Q-1:1" value="MMA8452QMMA8452Q-1:1"/>
-<part name="R1" library="SparkFun-Resistors" deviceset="10KOHM1/10W1%(0603)" device="0603" value="10k"/>
-<part name="C2" library="SparkFun-Capacitors" deviceset="4.7UF-6.3V-10%(0603)" device="0603" value="4.7uF"/>
+<part name="C1" library="SparkFun-Capacitors" deviceset="0.1UF" device="-0603-25V-(+80/-20%)" value="0.1uF"/>
+<part name="R1" library="SparkFun-Resistors" deviceset="10KOHM" device="-0603-1/10W-1%" value="10k"/>
+<part name="C2" library="SparkFun-Capacitors" deviceset="4.7UF" device="-0603-6.3V-(10%)" value="4.7uF"/>
 <part name="U2" library="SparkFun-PowerIC" deviceset="MIC5205" device="3.3V" value="MIC5205-3.3V"/>
-<part name="C3" library="SparkFun-Capacitors" deviceset="0.1UF-25V(+80/-20%)(0603)" device="" value="0.1uF"/>
+<part name="C3" library="SparkFun-Capacitors" deviceset="0.1UF" device="-0603-25V-(+80/-20%)" value="0.1uF"/>
 <part name="SUPPLY3" library="SparkFun-Aesthetics" deviceset="3.3V" device=""/>
 <part name="GND2" library="SparkFun-Aesthetics" deviceset="GND" device=""/>
@@
 <part name="SUPPLY6" library="SparkFun-PowerSymbols" deviceset="3.3V" device=""/>
 <part name="SUPPLY9" library="SparkFun-PowerSymbols" deviceset="3.3V" device=""/>
+<part name="LOGO4" library="SparkFun-Aesthetics" deviceset="SFE_LOGO_FLAME" device=".1_INCH"/>
+<part name="U1" library="SparkFun-Sensors" deviceset="MMA8452Q" device=""/>
 </parts>
 <sheets>
@@
 <text x="2.54" y="180.34" size="2.54" layer="94" font="vector">MMA8452Q Accelerometer</text>
 <text x="149.86" y="180.34" size="2.54" layer="94" font="vector">I2C Connections</text>
+<text x="2.54" y="86.36" size="1.27" layer="94" font="vector">VIN: 2.5-16V</text>
+<text x="58.42" y="114.3" size="1.778" layer="97" font="vector">7-bit Unshifted I2C Address: 0x1D</text>
 </plain>
 <instances>
@@
 <attribute name="VALUE" x="39.624" y="129.921" size="1.778" layer="96" font="vector"/>
 </instance>
-<instance part="U1" gate="G$1" x="81.28" y="137.16" smashed="yes">
-<attribute name="NAME" x="73.66" y="147.828" size="1.778" layer="95" font="vector"/>
-<attribute name="VALUE" x="73.66" y="124.714" size="1.778" layer="96" font="vector"/>
-</instance>
 <instance part="R1" gate="G$1" x="101.6" y="129.54" smashed="yes">
 <attribute name="NAME" x="97.79" y="131.0386" size="1.778" layer="95" font="vector"/>
@@
 <attribute name="VALUE" x="111.76" y="51.054" size="1.778" layer="96" font="vector" align="bottom-center"/>
 </instance>
+<instance part="LOGO4" gate="G$1" x="205.74" y="38.1" smashed="yes"/>
+<instance part="U1" gate="U1" x="81.28" y="137.16" smashed="yes">
+<attribute name="NAME" x="73.66" y="147.574" size="1.778" layer="95" font="vector"/>
+<attribute name="VALUE" x="73.66" y="126.746" size="1.778" layer="96" font="vector" align="top-left"/>
+</instance>
 </instances>
 <busses>
@@
 <net name="GND" class="0">
 <segment>
-<pinref part="U1" gate="G$1" pin="GND@2"/>
 <wire x1="71.12" y1="134.62" x2="68.58" y2="134.62" width="0.1524" layer="91"/>
 <wire x1="68.58" y1="134.62" x2="68.58" y2="132.08" width="0.1524" layer="91"/>
-<pinref part="U1" gate="G$1" pin="GND@0"/>
 <wire x1="68.58" y1="132.08" x2="68.58" y2="129.54" width="0.1524" layer="91"/>
 <wire x1="68.58" y1="129.54" x2="71.12" y2="129.54" width="0.1524" layer="91"/>
-<pinref part="U1" gate="G$1" pin="GND@1"/>
 <wire x1="71.12" y1="132.08" x2="68.58" y2="132.08" width="0.1524" layer="91"/>
 <junction x="68.58" y="132.08"/>
@@
 <pinref part="C1" gate="G$1" pin="2"/>
 <wire x1="38.1" y1="127" x2="38.1" y2="129.54" width="0.1524" layer="91"/>
+<pinref part="U1" gate="U1" pin="GND"/>
 </segment>
 <segment>
@@
 <net name="3.3V" class="0">
 <segment>
-<pinref part="U1" gate="G$1" pin="VDDIO"/>
 <wire x1="71.12" y1="142.24" x2="68.58" y2="142.24" width="0.1524" layer="91"/>
 <wire x1="68.58" y1="142.24" x2="68.58" y2="144.78" width="0.1524" layer="91"/>
-<pinref part="U1" gate="G$1" pin="VDD"/>
 <wire x1="68.58" y1="144.78" x2="71.12" y2="144.78" width="0.1524" layer="91"/>
 <junction x="68.58" y="142.24"/>
@@
 <wire x1="68.58" y1="149.86" x2="68.58" y2="144.78" width="0.1524" layer="91"/>
 <junction x="68.58" y="144.78"/>
+<pinref part="U1" gate="U1" pin="VDD"/>
 </segment>
 <segment>
@@
 <net name="ADDR" class="0">
 <segment>
-<pinref part="U1" gate="G$1" pin="SA0"/>
 <pinref part="R1" gate="G$1" pin="1"/>
 <wire x1="93.98" y1="129.54" x2="96.52" y2="129.54" width="0.1524" layer="91"/>
+<pinref part="U1" gate="U1" pin="SA0"/>
 </segment>
 </net>
@@
 <pinref part="C3" gate="G$1" pin="1"/>
 <wire x1="58.42" y1="137.16" x2="58.42" y2="139.7" width="0.1524" layer="91"/>
-<pinref part="U1" gate="G$1" pin="BYP"/>
 <wire x1="58.42" y1="139.7" x2="71.12" y2="139.7" width="0.1524" layer="91"/>
+<pinref part="U1" gate="U1" pin="BYP"/>
 </segment>
 </net>
@@
 <segment>
 <wire x1="96.52" y1="142.24" x2="93.98" y2="142.24" width="0.1524" layer="91"/>
-<pinref part="U1" gate="G$1" pin="SDA"/>
 <label x="96.52" y="142.24" size="1.27" layer="95" font="vector" xref="yes"/>
+<pinref part="U1" gate="U1" pin="SDA"/>
 </segment>
 </net>
@@
 </segment>
 <segment>
-<pinref part="U1" gate="G$1" pin="SCL"/>
 <wire x1="93.98" y1="144.78" x2="96.52" y2="144.78" width="0.1524" layer="91"/>
 <label x="96.52" y="144.78" size="1.27" layer="95" font="vector" xref="yes"/>
-</segment>
-</net>
+<pinref part="U1" gate="U1" pin="SCL"/>
+</segment>
+</net>

Commit message: post-review changes
Parts:
- removed LOGO1: LOGO-SFESK, SparkFun-Aesthetics:LOGO-SFESK
Other:
- note added: "Cut I2C Jumper to remove pullup resistors from the 5V I2C bus"
- note removed: "Cut I2C Jumper to remove pullup resistors from the I2C bus"
Changed lines of the file:
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@@
 <part name="GND1" library="SparkFun-Aesthetics" deviceset="GND" device=""/>
 <part name="FRAME1" library="SparkFun-Aesthetics" deviceset="FRAME-LETTER" device=""/>
-<part name="LOGO1" library="SparkFun-Aesthetics" deviceset="LOGO-SFE" device="SK"/>
 <part name="LOGO2" library="SparkFun-Aesthetics" deviceset="OSHW-LOGO" device="S"/>
 <part name="C1" library="SparkFun-Capacitors" deviceset="0.1UF" device="-0603-25V-(+80/-20%)" value="0.1uF"/>
@@
 <sheet>
 <plain>
-<text x="237.998" y="6.35" size="3.81" layer="94" font="vector">v14</text>
+<text x="237.744" y="7.874" size="2.54" layer="94" font="vector">v14</text>
 <text x="166.37" y="11.43" size="2.54" layer="94" font="vector">M. Hord</text>
 <text x="213.36" y="119.38" size="1.27" layer="97" font="vector">Top side
@@
 <text x="148.59" y="7.62" size="2.54" layer="94" font="vector">Revised by: Patrick Alberts, Andy England</text>
 <text x="106.68" y="58.42" size="1.27" layer="97" font="vector">Cut I2C Jumper to remove
-pullup resistors from the I2C bus</text>
+pullup resistors from the 5V I2C bus</text>
 <wire x1="147.32" y1="35.56" x2="147.32" y2="93.98" width="0.1524" layer="97" style="longdash"/>
 <wire x1="147.32" y1="93.98" x2="147.32" y2="185.42" width="0.1524" layer="97" style="longdash"/>
@@
 <attribute name="DRAWING_NAME" x="162.814" y="17.78" size="2.7432" layer="94" font="vector"/>
 </instance>
-<instance part="LOGO1" gate="G$1" x="241.3" y="17.78" smashed="yes"/>
 <instance part="LOGO2" gate="G$1" x="233.68" y="45.72" smashed="yes"/>
 <instance part="C1" gate="G$1" x="38.1" y="132.08" smashed="yes">
@@
 <net name="GND" class="0">
 <segment>
-<wire x1="71.12" y1="134.62" x2="68.58" y2="134.62" width="0.1524" layer="91"/>
-<wire x1="68.58" y1="134.62" x2="68.58" y2="132.08" width="0.1524" layer="91"/>
-<wire x1="68.58" y1="132.08" x2="68.58" y2="129.54" width="0.1524" layer="91"/>
 <wire x1="68.58" y1="129.54" x2="71.12" y2="129.54" width="0.1524" layer="91"/>
-<wire x1="71.12" y1="132.08" x2="68.58" y2="132.08" width="0.1524" layer="91"/>
-<junction x="68.58" y="132.08"/>
 <pinref part="GND1" gate="1" pin="GND"/>
 <wire x1="68.58" y1="124.46" x2="68.58" y2="127" width="0.1524" layer="91"/>
-<junction x="68.58" y="129.54"/>
 <pinref part="C3" gate="G$1" pin="2"/>
 <wire x1="68.58" y1="127" x2="68.58" y2="129.54" width="0.1524" layer="91"/>
@@
 <net name="3.3V" class="0">
 <segment>
-<wire x1="71.12" y1="142.24" x2="68.58" y2="142.24" width="0.1524" layer="91"/>
 <wire x1="68.58" y1="142.24" x2="68.58" y2="144.78" width="0.1524" layer="91"/>
 <wire x1="68.58" y1="144.78" x2="71.12" y2="144.78" width="0.1524" layer="91"/>
-<junction x="68.58" y="142.24"/>
 <wire x1="68.58" y1="142.24" x2="48.26" y2="142.24" width="0.1524" layer="91"/>
 <pinref part="C2" gate="G$1" pin="1"/>

Commit message: panelizing
Other:
- note added: "Revised by:Patrick Alberts, Andy England"
- note removed: "Revised by: Patrick Alberts, Andy England"
Changed lines of the file:
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@@
 connector-
 Female</text>
-<text x="148.59" y="7.62" size="2.54" layer="94" font="vector">Revised by: Patrick Alberts, Andy England</text>
+<text x="148.59" y="7.62" size="2.54" layer="94" font="vector">Revised by:Patrick Alberts, Andy England</text>
 <text x="106.68" y="58.42" size="1.27" layer="97" font="vector">Cut I2C Jumper to remove
 pullup resistors from the 5V I2C bus</text>
@@
 <attribute name="VALUE" x="186.944" y="102.616" size="1.778" layer="96" font="vector"/>
 </instance>
-<instance part="FID3" gate="G$1" x="193.04" y="38.1" smashed="yes"/>
-<instance part="FID1" gate="G$1" x="187.96" y="38.1" smashed="yes"/>
+<instance part="FID3" gate="G$1" x="246.38" y="25.4" smashed="yes"/>
+<instance part="FID1" gate="G$1" x="243.84" y="25.4" smashed="yes"/>
 <instance part="Q1" gate="NMOS" x="81.28" y="33.02" smashed="yes" rot="R270">
 <attribute name="NAME" x="81.28" y="27.94" size="1.778" layer="95" font="vector" rot="R270"/>
